File: EagleFiles/amplifier.brd (EAGLE design)
At the start: 100 x 94 mm, 59 parts

Commit message: final version
Parts:
- C14: value 680p -> 1.2nF
- R24: value 5.6K -> 3.3K
- moved R1 2.82 mm to (23.5, 37.7)
- moved EF86 1.27 mm to (16.3, 50.9)
- moved C11 0.81 mm to (30.6, 68.6), turned to 90 degrees
- moved R19 0.08 mm to (87.4, 54.3), flipped to the bottom, turned to 180 degrees
- flipped R18 to the bottom, turned to 180 degrees
Connections:
- net KT88 renamed KT88ANODE_1
- net KT88_2 renamed KT88ANODE_2
- net N$11 renamed KT88GRID_1
- net N$15 renamed KT88GRID_2
- net N$18 renamed KT88KATHODE_2
- net N$19 renamed KT88KATHODE_1
- net N$31 renamed ECC82FILL-
- net N$32 renamed ECC82FILL+
- net N$33 renamed KT88FILLAMENT-
- net N$34 renamed KT88FILLAMENT+
- net N$37 renamed EF86FILL+
- net N$38 renamed EF86FILL-
Routing:
- net KT88GRID_1: track 22.3 -> 33.4 mm
- net DIFFOUTPUT_N: track 64.7 -> 73.8 mm
- net DIFFOUTPUT_P: track 70.4 -> 74.9 mm
- net KT88ANODE_1: track 63.4 -> 60.6 mm
- net N$4: track 69.8 -> 72.1 mm
- net GND: track 21.7 -> 23.9 mm
- net N$13: track 32.3 -> 30.0 mm
- net KT88GRID_2: track 34.4 -> 36.0 mm
- net N$3: track 49.6 -> 50.5 mm
- net EF86FILL-: track 19.7 -> 18.8 mm
- net N$21: track 27.3 -> 26.6 mm
- net N$23: track 37.1 -> 37.8 mm
Other:
- board text added: "12.6V_ECC82"
- board text added: "6.3V KT88+"
- board text added: "6.3_KT88 -"
- board text added: "C1"
- board text added: "C12"
- board text added: "C13"
- board text added: "C14"
- board text added: "C2"
- board text added: "C3"
- board text added: "C4"
- board text added: "C5"
- board text added: "C6"
- board text added: "FEEDBACK 4OHM"
- board text added: "FEEDBACK 8OHM"
- board text added: "GND_RCA"
- board text added: "INPUT"
- board text added: "KT88 Anode"
- board text added: "KT88 Grid"
- board text added: "R22"
- board text added: "R23"
- board text added: "R24"
- board text added: "Tosis V1.2"
- board text removed: "12.6V ECC82"
- board text removed: "6.3_KT88"
- board text removed: "FEEDBACK"
- board text removed: "KT88"
- board text removed: "KT88_OUTPUT"
- board text removed: "KT88_TRAFO"
- board text removed: "Tosis V 1.0"
- board text removed: "VSS"
