File: EagleFiles/amplifier.sch (EAGLE design)
At the start: 52 parts, among them X1 736880-49

Commit message: Fix Feedback
Connections:
- removed net N$5: C2.-, R6.2, R7.1
- new net N$35: C2.+, EF86G$1.PK, R6.1
- new net N$36: EF86G$1.PBG
- net N$3: now also C2.-, R6.2, R7.1; no longer C2.+, EF86G$1.PBG, EF86G$1.PK, R6.1
Other:
- moved on the sheet: C7, R8
Changed lines of the file:
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@@
 <instance part="R3" gate="G$1" x="45.72" y="81.28"/>
 <instance part="R7" gate="G$1" x="35.56" y="20.32" rot="R270"/>
-<instance part="R8" gate="G$1" x="50.8" y="43.18"/>
+<instance part="R8" gate="G$1" x="48.26" y="27.94"/>
 <instance part="R6" gate="G$1" x="35.56" y="38.1" rot="R270"/>
 <instance part="R16" gate="G$1" x="76.2" y="53.34" rot="R90"/>
@@
 <instance part="C9" gate="G$1" x="134.62" y="68.58" rot="R90"/>
 <instance part="C6" gate="G$1" x="58.42" y="66.04"/>
-<instance part="C7" gate="G$1" x="48.26" y="30.48" rot="R90"/>
+<instance part="C7" gate="G$1" x="48.26" y="17.78" rot="R90"/>
 <instance part="GND1" gate="1" x="7.62" y="22.86"/>
 <instance part="GND2" gate="1" x="35.56" y="10.16"/>
@@
 </segment>
 </net>
-<net name="N$3" class="0">
-<segment>
-<pinref part="EF86" gate="G$1" pin="PK"/>
-<wire x1="35.56" y1="43.18" x2="45.72" y2="43.18" width="0.1524" layer="91"/>
-<wire x1="45.72" y1="43.18" x2="45.72" y2="58.42" width="0.1524" layer="91"/>
-<pinref part="EF86" gate="G$1" pin="PBG"/>
-<wire x1="45.72" y1="58.42" x2="40.64" y2="58.42" width="0.1524" layer="91"/>
-<pinref part="R6" gate="G$1" pin="1"/>
-<junction x="35.56" y="43.18"/>
-<pinref part="R8" gate="G$1" pin="1"/>
-<junction x="45.72" y="43.18"/>
-<pinref part="C7" gate="G$1" pin="1"/>
-<wire x1="45.72" y1="30.48" x2="45.72" y2="43.18" width="0.1524" layer="91"/>
-<pinref part="C2" gate="G$1" pin="+"/>
-<wire x1="20.32" y1="40.64" x2="20.32" y2="43.18" width="0.1524" layer="91"/>
-<wire x1="20.32" y1="43.18" x2="35.56" y2="43.18" width="0.1524" layer="91"/>
-</segment>
-</net>
 <net name="N$4" class="0">
 <segment>
@@
 <wire x1="66.04" y1="60.96" x2="58.42" y2="60.96" width="0.1524" layer="91"/>
 <junction x="58.42" y="60.96"/>
-</segment>
-</net>
-<net name="N$5" class="0">
-<segment>
-<pinref part="R6" gate="G$1" pin="2"/>
-<pinref part="R7" gate="G$1" pin="1"/>
-<wire x1="35.56" y1="25.4" x2="35.56" y2="33.02" width="0.1524" layer="91"/>
-<pinref part="C2" gate="G$1" pin="-"/>
-<wire x1="20.32" y1="33.02" x2="35.56" y2="33.02" width="0.1524" layer="91"/>
-<junction x="35.56" y="33.02"/>
 </segment>
 </net>
@@
 <net name="N$12" class="0">
 <segment>
-<pinref part="R8" gate="G$1" pin="2"/>
-<wire x1="55.88" y1="43.18" x2="55.88" y2="30.48" width="0.1524" layer="91"/>
-<pinref part="C7" gate="G$1" pin="2"/>
-<wire x1="55.88" y1="30.48" x2="53.34" y2="30.48" width="0.1524" layer="91"/>
-<wire x1="55.88" y1="30.48" x2="55.88" y2="0" width="0.1524" layer="91"/>
-<junction x="55.88" y="30.48"/>
-<wire x1="55.88" y1="0" x2="226.06" y2="0" width="0.1524" layer="91"/>
+<wire x1="53.34" y1="0" x2="226.06" y2="0" width="0.1524" layer="91"/>
 <wire x1="226.06" y1="0" x2="226.06" y2="48.26" width="0.1524" layer="91"/>
 <pinref part="FEEDBACK" gate="1" pin="P"/>
+<pinref part="C7" gate="G$1" pin="2"/>
+<wire x1="53.34" y1="0" x2="53.34" y2="17.78" width="0.1524" layer="91"/>
+<pinref part="R8" gate="G$1" pin="2"/>
+<wire x1="53.34" y1="17.78" x2="53.34" y2="27.94" width="0.1524" layer="91"/>
+<junction x="53.34" y="17.78"/>
+<junction x="53.34" y="27.94"/>
 </segment>
 </net>
@@
 </segment>
 </net>
+<net name="N$35" class="0">
+<segment>
+<pinref part="EF86" gate="G$1" pin="PK"/>
+<pinref part="R6" gate="G$1" pin="1"/>
+<junction x="35.56" y="43.18"/>
+<wire x1="20.32" y1="43.18" x2="35.56" y2="43.18" width="0.1524" layer="91"/>
+<pinref part="C2" gate="G$1" pin="+"/>
+<wire x1="20.32" y1="40.64" x2="20.32" y2="43.18" width="0.1524" layer="91"/>
+</segment>
+</net>
+<net name="N$36" class="0">
+<segment>
+<pinref part="EF86" gate="G$1" pin="PBG"/>
+<wire x1="45.72" y1="58.42" x2="40.64" y2="58.42" width="0.1524" layer="91"/>
+</segment>
+</net>
+<net name="N$3" class="0">
+<segment>
+<pinref part="C7" gate="G$1" pin="1"/>
+<pinref part="R8" gate="G$1" pin="1"/>
+<wire x1="45.72" y1="17.78" x2="43.18" y2="17.78" width="0.1524" layer="91"/>
+<wire x1="43.18" y1="17.78" x2="43.18" y2="27.94" width="0.1524" layer="91"/>
+<wire x1="43.18" y1="27.94" x2="43.18" y2="33.02" width="0.1524" layer="91"/>
+<junction x="43.18" y="27.94"/>
+<pinref part="R6" gate="G$1" pin="2"/>
+<pinref part="R7" gate="G$1" pin="1"/>
+<wire x1="35.56" y1="25.4" x2="35.56" y2="33.02" width="0.1524" layer="91"/>
+<pinref part="C2" gate="G$1" pin="-"/>
+<wire x1="20.32" y1="33.02" x2="35.56" y2="33.02" width="0.1524" layer="91"/>
+<junction x="35.56" y="33.02"/>
+<wire x1="43.18" y1="33.02" x2="35.56" y2="33.02" width="0.1524" layer="91"/>
+<junction x="45.72" y="17.78"/>
+</segment>
+</net>

Commit message: last not good design.
Parts:
- removed VSS: (no value), jumper:JP1E
- removed X1: 736880-49, con-conrad:736880-49
- added GND_, INPUT: (no value), wirepad:2,54/1,0
- C1: device resistor:CPOL-EUE10-20 -> rcl:CPOL-EUE5-13
- C12: value 100mF/100V -> 100u/100V; device rcl:CPOL-EUE7.5-18 -> rcl:CPOL-EUE5-10.5
- C2: value 10m/25V -> 10u/25V; device resistor:CPOL-EUE10-20 -> rcl:CPOL-EUE5-8.5
- C3: value 10m -> 10u/450V; device resistor:CPOL-EUE10-20 -> rcl:CPOL-EUE5-13
- C4: value 100uF/100V -> 100u/100V; device rcl:CPOL-EUE7.5-18 -> rcl:CPOL-EUE5-10.5
- C5: value 100nF -> 100n
- U$2, U$3: value KT88 -> KT88OKTAL1; device Tubes_all:KT88 -> tubes_stockes:KT88OKTAL1
Connections:
- removed net N$30: VSS.1, VSS.2
- removed net N$35: C2.+, EF86G$1.PK, R6.1
- net GND: now also GND_.P; no longer X1.1
- net N$1: now also INPUT.P; no longer X1.2
- net N$36: now also C2.+, EF86G$1.PK, R6.1
Other:
- note removed: "380 V"

Commit message: back to old design, bigger dimensions and 2 feedbacks.
Parts:
- removed FEEDBACK: (no value), wirepad:2,54/1,1
- removed GND_: (no value), wirepad:2,54/1,0
- removed U$1: (no value), Bourns:DUALPOTAUDIO
- added 6.3_KTGND: 6.3 V, jumper:JP1E
- added C13: 100nF, rcl:C-EUC0805K
- added C14: 680p, capacitor-wima:C5/5.5
- added FEEDBACK4OHM, FEEDBACK8OHM: (no value), wirepad:2,54/1,1
- added GND_RCA: WIREPAD2,15/1,0, wirepad:WIREPAD2,15/1,0
- added POT: 100K, Bourns:DUALPOTAUDIO
- added R22, R23: 470/5W, resistor_mod:R-EU_0617/5V
- added R24: 5.6K, rcl:R-EU_R0805
- C1, C3: device rcl:CPOL-EUE5-13 -> rcl:CPOL-EUE5-10.5
- C10, C11, C5: value 100n -> 100nF; device resistor:C-EU102-054X133 -> capacitor-wima:C7.5/3
- C12, C4: value 100u/100V -> 100uF/100V; device rcl:CPOL-EUE5-10.5 -> rcl:CPOL-EUE3.5-10
- C2: device rcl:CPOL-EUE5-8.5 -> rcl:CPOL-EUE3.5-10
- C6, C7: device resistor:C-EU050-045X075 -> capacitor-wima:C5/5.5
- C8, C9: value 220n -> 220nF; device resistor:C-EU102-054X133 -> capacitor-wima:C7.5/3
- INPUT: value (none) -> WIREPAD2,15/1,0; device wirepad:2,54/1,0 -> wirepad:WIREPAD2,15/1,0
- R13, R4: value 220/5W -> 470/5W; device rcl:R-EU_0817/7V -> resistor_mod:R-EU_0617/5V
Connections:
- net N$10 renamed DIFFOUTPUT_P
- net N$14 renamed DIFFOUTPUT_N
- removed net N$36: C2.+, EF86G$1.PBG, EF86G$1.PK, R6.1
- removed net N56: KT88_OUTPUT.2, R18.2
- new net N$10: C14.2, C2.-, C7.1, R24.2, R6.1, R7.1, R8.1
- new net N$14: C14.1, FEEDBACK4OHM.P, R24.1
- new net N$35: C13.1, JMP1-0R.2
- new net N$56: KT88_TRAFO.2, R18.2
- net GND: now also GND_RCA.P, POT.R1_1, POT.R2_1, POT.SW0, POT.SW1, R22.2, R23.2; no longer GND_.P, U$1.R1_1, U$1.R2_1, U$1.SW0, U$1.SW1
- net KT88: now also KT88_OUTPUT.1; no longer KT88_TRAFO.1
- net KT88_2: now also KT88_OUTPUT.2; no longer KT88_TRAFO.2
- net N$12: now also FEEDBACK8OHM.P; no longer FEEDBACK.P
- net N$18: now also R23.1
- net N$19: now also R22.1
- net N$2: now also C13.2; no longer JMP1-0R.2
- net N$21: now also POT.R1_2; no longer U$1.R1_2
- net N$22: now also POT.R1_3; no longer U$1.R1_3
- net N$26: now also POT.R2_2; no longer U$1.R2_2
- net N$27: now also KT88_TRAFO.1; no longer KT88_OUTPUT.1
- net N$28: now also POT.R2_3; no longer U$1.R2_3
- net N$3: now also C2.+, EF86G$1.PBG, EF86G$1.PK; no longer C2.-, C7.1, R7.1, R8.1
- net N$33: now also 6.3_KTGND.1, 6.3_KTGND.2; no longer 6.3_KT88.1
- net N$34: now also 6.3_KT88.1
Other:
- note removed: "100K"
- moved on the sheet: C7, R6, R8

Commit message: final version
Parts:
- C14: value 680p -> 1.2nF
- R24: value 5.6K -> 3.3K
Connections:
- net KT88 renamed KT88ANODE_1
- net KT88_2 renamed KT88ANODE_2
- net N$11 renamed KT88GRID_1
- net N$15 renamed KT88GRID_2
- net N$18 renamed KT88KATHODE_2
- net N$19 renamed KT88KATHODE_1
- net N$31 renamed ECC82FILL-
- net N$32 renamed ECC82FILL+
- net N$33 renamed KT88FILLAMENT-
- net N$34 renamed KT88FILLAMENT+
- net N$37 renamed EF86FILL+
- net N$38 renamed EF86FILL-
Other:
- moved on the sheet: C11, ECC82B, GND_RCA, INPUT, R15
